File: karta_stm/file5F905B55.sch (KiCad schematic (older format))
At the start: 35 parts, among them J1 Conn_01x02_Female, J2 Conn_01x06_Male, J3 Conn_01x05_Female, J7 Conn_01x03_Male, SW1 SW_Push, U1 STM32L4P5RET6, U2 MCP2562-H-SN, Y1 16MHz

Commit message: Update pcb
Parts:
- C1, C2: footprint Capacitor_SMD:C_0805_2012Metric_Pad1.15x1.40mm_HandSolder -> Capacitor_SMD:C_0805_2012Metric
- C10, C12, C3: footprint Capacitor_SMD:C_1206_3216Metric_Pad1.42x1.75mm_HandSolder -> Capacitor_SMD:C_1206_3216Metric
- C11: footprint Capacitor_SMD:C_1206_3216Metric_Pad1.42x1.75mm_HandSolder -> Capacitor_SMD:CP_Elec_4x5.7
- C9: footprint Capacitor_Tantalum_SMD:CP_EIA-6032-15_Kemet-U_Pad2.25x2.35mm_HandSolder -> Capacitor_Tantalum_SMD:CP_EIA-6032-15_Kemet-U
- D11: footprint Diode_SMD:D_1210_3225Metric_Pad1.42x2.65mm_HandSolder -> Diode_SMD:D_1210_3225Metric
- R1: footprint Resistor_SMD:R_1206_3216Metric_Pad1.42x1.75mm_HandSolder -> Resistor_SMD:R_1206_3216Metric
- R2, R3, R48: footprint Resistor_SMD:R_1206_3216Metric_Pad1.42x1.75mm_HandSolder -> Resistor_SMD:R_0805_2012Metric
- SW1: footprint Button_Switch_SMD:SW_Push_1P1T_NO_6x6mm_H9.5mm -> Resistor_SMD:R_0805_2012Metric
Changed lines of the file:
@@
 F 0 "C12" H 8965 1196 50  0000 L CNN
 F 1 "100nF" H 8965 1105 50  0000 L CNN
-F 2 "Capacitor_SMD:C_1206_3216Metric_Pad1.42x1.75mm_HandSolder" H 8888 1000 50  0001 C CNN
+F 2 "Capacitor_SMD:C_1206_3216Metric" H 8888 1000 50  0001 C CNN
 F 3 "~" H 8850 1150 50  0001 C CNN
 	1    8850 1150
@@
 F 0 "C3" H 6615 3096 50  0000 L CNN
 F 1 "0.1uF" H 6615 3005 50  0000 L CNN
-F 2 "Capacitor_SMD:C_1206_3216Metric_Pad1.42x1.75mm_HandSolder" H 6538 2900 50  0001 C CNN
+F 2 "Capacitor_SMD:C_1206_3216Metric" H 6538 2900 50  0001 C CNN
 F 3 "~" H 6500 3050 50  0001 C CNN
 	1    6500 3050
@@
 F 0 "SW1" H 6400 3985 50  0000 C CNN
 F 1 "SW_Push" H 6400 3894 50  0000 C CNN
-F 2 "Button_Switch_SMD:SW_Push_1P1T_NO_6x6mm_H9.5mm" H 6400 3900 50  0001 C CNN
+F 2 "Resistor_SMD:R_0805_2012Metric" H 6400 3900 50  0001 C CNN
 F 3 "~" H 6400 3900 50  0001 C CNN
 	1    6400 3700
@@
 F 0 "R1" V 5793 3050 50  0000 C CNN
 F 1 "0R" V 5884 3050 50  0000 C CNN
-F 2 "Resistor_SMD:R_1206_3216Metric_Pad1.42x1.75mm_HandSolder" V 5930 3050 50  0001 C CNN
+F 2 "Resistor_SMD:R_1206_3216Metric" V 5930 3050 50  0001 C CNN
 F 3 "~" H 6000 3050 50  0001 C CNN
 	1    6000 3050
@@
 F 0 "R2" V 5893 7050 50  0000 C CNN
 F 1 "10k Ohm" V 5984 7050 50  0000 C CNN
-F 2 "Resistor_SMD:R_1206_3216Metric_Pad1.42x1.75mm_HandSolder" V 6030 7050 50  0001 C CNN
+F 2 "Resistor_SMD:R_0805_2012Metric" V 6030 7050 50  0001 C CNN
 F 3 "~" H 6100 7050 50  0001 C CNN
 	1    6100 7050
@@
 F 0 "C2" V 4052 7400 50  0000 C CNN
 F 1 "20pF" V 3961 7400 50  0000 C CNN
-F 2 "Capacitor_SMD:C_0805_2012Metric_Pad1.15x1.40mm_HandSolder" H 3838 7250 50  0001 C CNN
+F 2 "Capacitor_SMD:C_0805_2012Metric" H 3838 7250 50  0001 C CNN
 F 3 "~" H 3800 7400 50  0001 C CNN
 	1    3800 7400
@@
 F 0 "C1" V 3548 7000 50  0000 C CNN
 F 1 "20pF" V 3639 7000 50  0000 C CNN
-F 2 "Capacitor_SMD:C_0805_2012Metric_Pad1.15x1.40mm_HandSolder" H 3838 6850 50  0001 C CNN
+F 2 "Capacitor_SMD:C_0805_2012Metric" H 3838 6850 50  0001 C CNN
 F 3 "~" H 3800 7000 50  0001 C CNN
 	1    3800 7000
@@
 F 0 "R3" H 10370 2146 50  0000 L CNN
 F 1 "120 Ohm" H 10370 2055 50  0000 L CNN
-F 2 "Resistor_SMD:R_1206_3216Metric_Pad1.42x1.75mm_HandSolder" V 10230 2100 50  0001 C CNN
+F 2 "Resistor_SMD:R_0805_2012Metric" V 10230 2100 50  0001 C CNN
 F 3 "~" H 10300 2100 50  0001 C CNN
 	1    10300 2100
@@
 F 0 "D11" V 2846 7470 50  0000 R CNN
 F 1 "D" V 2755 7470 50  0000 R CNN
-F 2 "Diode_SMD:D_1210_3225Metric_Pad1.42x2.65mm_HandSolder" H 2800 7550 50  0001 C CNN
+F 2 "Diode_SMD:D_1210_3225Metric" H 2800 7550 50  0001 C CNN
 F 3 "~" H 2800 7550 50  0001 C CNN
 	1    2800 7550
@@
 F 0 "R48" H 3170 7596 50  0000 L CNN
 F 1 "1kOhm" H 3170 7505 50  0000 L CNN
-F 2 "Resistor_SMD:R_1206_3216Metric_Pad1.42x1.75mm_HandSolder" V 3030 7550 50  0001 C CNN
+F 2 "Resistor_SMD:R_0805_2012Metric" V 3030 7550 50  0001 C CNN
 F 3 "~" H 3100 7550 50  0001 C CNN
 	1    3100 7550
@@
 F 0 "C11" H 7868 5346 50  0000 L CNN
 F 1 "1uF" H 7868 5255 50  0000 L CNN
-F 2 "Capacitor_SMD:C_1206_3216Metric_Pad1.42x1.75mm_HandSolder" H 7788 5150 50  0001 C CNN
+F 2 "Capacitor_SMD:CP_Elec_4x5.7" H 7788 5150 50  0001 C CNN
 F 3 "~" H 7750 5300 50  0001 C CNN
 	1    7750 5300
@@
 F 0 "C10" H 7465 5346 50  0000 L CNN
 F 1 "10nF" H 7465 5255 50  0000 L CNN
-F 2 "Capacitor_SMD:C_1206_3216Metric_Pad1.42x1.75mm_HandSolder" H 7388 5150 50  0001 C CNN
+F 2 "Capacitor_SMD:C_1206_3216Metric" H 7388 5150 50  0001 C CNN
 F 3 "~" H 7350 5300 50  0001 C CNN
 	1    7350 5300
@@
 F 0 "C9" H 7068 5346 50  0000 L CNN
 F 1 "4,7uF" H 7068 5255 50  0000 L CNN
-F 2 "Capacitor_Tantalum_SMD:CP_EIA-6032-15_Kemet-U_Pad2.25x2.35mm_HandSolder" H 6988 5150 50  0001 C CNN
+F 2 "Capacitor_Tantalum_SMD:CP_EIA-6032-15_Kemet-U" H 6988 5150 50  0001 C CNN
 F 3 "~" H 6950 5300 50  0001 C CNN
 	1    6950 5300
