File: karta_stm/file5F916EBD.sch (KiCad schematic (older format))
At the start: 18 parts, among them J4 Conn_01x02_Female, U3 LM2596S-5, U4 LD1117S33TR_SOT223

Commit message: Update pcb
Parts:
- removed U4: LD1117S33TR_SOT223, Package_TO_SOT_SMD:SOT-223-3_TabPin2, symbol karta_stm-rescue:LD1117S33TR_SOT223-Regulator_Linear
- added U4: LM1117-3.3, Package_TO_SOT_SMD:SOT-223-3_TabPin2, symbol Regulator_Linear:LM1117-3.3
- D12: footprint Diode_SMD:D_1210_3225Metric_Pad1.42x2.65mm_HandSolder -> Diode_SMD:D_1210_3225Metric
- D3: value D_Schottky -> SS24T3G
- F1: footprint Fuse:Fuse_2920_7451Metric_Pad2.10x5.45mm_HandSolder -> Fuse:Fuse_1206_3216Metric_Pad1.42x1.75mm_HandSolder
- R49: value 1kOhm -> 5kOhm; footprint Resistor_SMD:R_1206_3216Metric_Pad1.42x1.75mm_HandSolder -> Resistor_SMD:R_0805_2012Metric
Changed lines of the file:
@@
 P 2700 1500
 F 0 "D3" H 2700 1283 50  0000 C CNN
-F 1 "D_Schottky" H 2700 1374 50  0000 C CNN
+F 1 "SS24T3G" H 2700 1374 50  0000 C CNN
 F 2 "Diode_SMD:D_SMB" H 2700 1500 50  0001 C CNN
 F 3 "~" H 2700 1500 50  0001 C CNN
@@
 	700  1500 850  1500
 $Comp
-L karta_stm-rescue:LD1117S33TR_SOT223-Regulator_Linear U4
-U 1 1 5F923BA6
-P 3200 2750
-F 0 "U4" H 3200 2992 50  0000 C CNN
-F 1 "LD1117S33TR_SOT223" H 3200 2901 50  0000 C CNN
-F 2 "Package_TO_SOT_SMD:SOT-223-3_TabPin2" H 3200 2950 50  0001 C CNN
-F 3 "http://www.st.com/st-web-ui/static/active/en/resource/technical/document/datasheet/CD00000544.pdf" H 3300 2500 50  0001 C CNN
-	1    3200 2750
-	1    0    0    -1
-$EndComp
-$Comp
 L karta_stm-rescue:+5V-power #PWR022
 U 1 1 5F924B9A
@@
 Wire Wire Line
 	2600 2750 2900 2750
-Wire Wire Line
-	3800 3050 3200 3050
-Connection ~ 3200 3050
-Wire Wire Line
-	3200 3050 2600 3050
 $Comp
 L karta_stm-rescue:GND-power #PWR026
@@
 F 0 "D12" V 4446 2820 50  0000 R CNN
 F 1 "D" V 4355 2820 50  0000 R CNN
-F 2 "Diode_SMD:D_1210_3225Metric_Pad1.42x2.65mm_HandSolder" H 4400 2900 50  0001 C CNN
+F 2 "Diode_SMD:D_1210_3225Metric" H 4400 2900 50  0001 C CNN
 F 3 "~" H 4400 2900 50  0001 C CNN
 	1    4400 2900
@@
 P 4400 3200
 F 0 "R49" H 4470 3246 50  0000 L CNN
-F 1 "1kOhm" H 4470 3155 50  0000 L CNN
-F 2 "Resistor_SMD:R_1206_3216Metric_Pad1.42x1.75mm_HandSolder" V 4330 3200 50  0001 C CNN
+F 1 "5kOhm" H 4470 3155 50  0000 L CNN
+F 2 "Resistor_SMD:R_0805_2012Metric" V 4330 3200 50  0001 C CNN
 F 3 "~" H 4400 3200 50  0001 C CNN
 	1    4400 3200
@@
 Wire Wire Line
 	3150 3350 3150 3400
-Wire Wire Line
-	3200 3100 3200 3350
 Connection ~ 3200 3350
 Wire Wire Line
@@
 F 0 "F1" V 803 1500 50  0000 C CNN
 F 1 "200mA" V 894 1500 50  0000 C CNN
-F 2 "Fuse:Fuse_2920_7451Metric_Pad2.10x5.45mm_HandSolder" V 930 1500 50  0001 C CNN
+F 2 "Fuse:Fuse_1206_3216Metric_Pad1.42x1.75mm_HandSolder" V 930 1500 50  0001 C CNN
 F 3 "~" H 1000 1500 50  0001 C CNN
 	1    1000 1500
@@
 	-1   0    0    1
 $EndComp
+$Comp
+L Regulator_Linear:LM1117-3.3 U4
+U 1 1 60BAD92C
+P 3200 2750
+F 0 "U4" H 3200 2992 50  0000 C CNN
+F 1 "LM1117-3.3" H 3200 2901 50  0000 C CNN
+F 2 "Package_TO_SOT_SMD:SOT-223-3_TabPin2" H 3200 2750 50  0001 C CNN
+F 3 "http://www.ti.com/lit/ds/symlink/lm1117.pdf" H 3200 2750 50  0001 C CNN
+	1    3200 2750
+	1    0    0    -1
+$EndComp
+Wire Wire Line
+	2600 3050 3200 3050
+Connection ~ 3200 3050
+Wire Wire Line
+	3200 3050 3800 3050
+Wire Wire Line
+	3200 3050 3200 3350
 $EndSCHEMATC
