File: karta_stm/file5F944891.sch (KiCad schematic (older format))
At the start: 36 parts, among them J5 Conn_01x05_Female, U5 MCP6001x-LT, U6 MCP6001x-LT, U7 MCP6001x-LT, U8 MCP6001x-LT, U9 MCP6001x-LT

Commit message: Update pcb
Parts:
- C18, C19, C20, C21, C22: footprint Capacitor_SMD:C_1206_3216Metric_Pad1.42x1.75mm_HandSolder -> Capacitor_SMD:C_1206_3216Metric
- R10, R11, R12, R13, R14, R15, R16, R17, R18, R19, R20, R21, R22, R23, R4, R5, R6, R7, R8, R9: footprint Resistor_SMD:R_1206_3216Metric_Pad1.42x1.75mm_HandSolder -> Resistor_SMD:R_0805_2012Metric
