File: karta_stm/file5F94992F.sch (KiCad schematic (older format))
At the start: 13 parts, among them J6 Conn_01x04_Female, U10 EL817, U11 EL817, U12 EL817, U13 EL817

Commit message: Update pcb
Parts:
- R24, R25, R26, R27, R28, R29, R30, R31: footprint Resistor_SMD:R_1206_3216Metric_Pad1.42x1.75mm_HandSolder -> Resistor_SMD:R_0805_2012Metric
Changed lines of the file:
@@
 F 0 "R25" H 2870 1896 50  0000 L CNN
 F 1 "R" H 2870 1805 50  0000 L CNN
-F 2 "Resistor_SMD:R_1206_3216Metric_Pad1.42x1.75mm_HandSolder" V 2730 1850 50  0001 C CNN
+F 2 "Resistor_SMD:R_0805_2012Metric" V 2730 1850 50  0001 C CNN
 F 3 "~" H 2800 1850 50  0001 C CNN
 	1    2800 1850
@@
 F 0 "R26" V 4557 1500 50  0000 C CNN
 F 1 "10k" V 4466 1500 50  0000 C CNN
-F 2 "Resistor_SMD:R_1206_3216Metric_Pad1.42x1.75mm_HandSolder" V 4280 1500 50  0001 C CNN
+F 2 "Resistor_SMD:R_0805_2012Metric" V 4280 1500 50  0001 C CNN
 F 3 "~" H 4350 1500 50  0001 C CNN
 	1    4350 1500
@@
 F 0 "R27" H 5420 1896 50  0000 L CNN
 F 1 "R" H 5420 1805 50  0000 L CNN
-F 2 "Resistor_SMD:R_1206_3216Metric_Pad1.42x1.75mm_HandSolder" V 5280 1850 50  0001 C CNN
+F 2 "Resistor_SMD:R_0805_2012Metric" V 5280 1850 50  0001 C CNN
 F 3 "~" H 5350 1850 50  0001 C CNN
 	1    5350 1850
@@
 F 0 "R28" V 7007 1500 50  0000 C CNN
 F 1 "10k" V 6916 1500 50  0000 C CNN
-F 2 "Resistor_SMD:R_1206_3216Metric_Pad1.42x1.75mm_HandSolder" V 6730 1500 50  0001 C CNN
+F 2 "Resistor_SMD:R_0805_2012Metric" V 6730 1500 50  0001 C CNN
 F 3 "~" H 6800 1500 50  0001 C CNN
 	1    6800 1500
@@
 F 0 "R29" H 7920 1896 50  0000 L CNN
 F 1 "R" H 7920 1805 50  0000 L CNN
-F 2 "Resistor_SMD:R_1206_3216Metric_Pad1.42x1.75mm_HandSolder" V 7780 1850 50  0001 C CNN
+F 2 "Resistor_SMD:R_0805_2012Metric" V 7780 1850 50  0001 C CNN
 F 3 "~" H 7850 1850 50  0001 C CNN
 	1    7850 1850
@@
 F 0 "R30" V 9507 1500 50  0000 C CNN
 F 1 "10k" V 9416 1500 50  0000 C CNN
-F 2 "Resistor_SMD:R_1206_3216Metric_Pad1.42x1.75mm_HandSolder" V 9230 1500 50  0001 C CNN
+F 2 "Resistor_SMD:R_0805_2012Metric" V 9230 1500 50  0001 C CNN
 F 3 "~" H 9300 1500 50  0001 C CNN
 	1    9300 1500
@@
 F 0 "R31" H 10370 1896 50  0000 L CNN
 F 1 "R" H 10370 1805 50  0000 L CNN
-F 2 "Resistor_SMD:R_1206_3216Metric_Pad1.42x1.75mm_HandSolder" V 10230 1850 50  0001 C CNN
+F 2 "Resistor_SMD:R_0805_2012Metric" V 10230 1850 50  0001 C CNN
 F 3 "~" H 10300 1850 50  0001 C CNN
 	1    10300 1850
@@
 F 0 "R24" V 2107 1500 50  0000 C CNN
 F 1 "10k" V 2016 1500 50  0000 C CNN
-F 2 "Resistor_SMD:R_1206_3216Metric_Pad1.42x1.75mm_HandSolder" V 1830 1500 50  0001 C CNN
+F 2 "Resistor_SMD:R_0805_2012Metric" V 1830 1500 50  0001 C CNN
 F 3 "~" H 1900 1500 50  0001 C CNN
 	1    1900 1500
