File: karta_stm/file5F96D222.sch (KiCad schematic (older format))
At the start: 33 parts, among them Q1 BC817, Q10 BC817, Q11 Q_PMOS_DGS, Q12 Q_NMOS_DGS, Q13 BC817, Q14 Q_PMOS_DGS, Q15 Q_NMOS_DGS, Q2 Q_PMOS_DGS, Q3 Q_NMOS_DGS, Q4 BC817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

Commit message: changed
Parts:
- R41: value 100k -> 10k
Changed lines of the file:
@@
 EESchema Schematic File Version 4
-LIBS:karta_stm-cache
-EELAYER 29 0
+EELAYER 30 0
 EELAYER END
 $Descr A4 11693 8268
@@
 P 4400 900
 F 0 "R41" H 4470 946 50  0000 L CNN
-F 1 "100k" H 4470 855 50  0000 L CNN
+F 1 "10k" H 4470 855 50  0000 L CNN
 F 2 "Resistor_SMD:R_1206_3216Metric_Pad1.42x1.75mm_HandSolder" V 4330 900 50  0001 C CNN
 F 3 "~" H 4400 900 50  0001 C CNN

Commit message: Update pcb
Parts:
- F2: footprint Fuse:Fuse_2920_7451Metric_Pad2.10x5.45mm_HandSolder -> Fuse:Fuse_1206_3216Metric_Pad1.42x1.75mm_HandSolder
- Q11, Q14, Q5, Q8: value Q_PMOS_DGS -> BSS84AKW.115; footprint Package_TO_SOT_SMD:SOT-23W_Handsoldering -> Package_TO_SOT_SMD:SOT-23; symbol karta_stm-rescue:Q_PMOS_DGS-Device -> Device:Q_PMOS_GSD
- Q12, Q15, Q3, Q6, Q9: value Q_NMOS_DGS -> BSS138W; footprint Package_TO_SOT_SMD:SOT-23W_Handsoldering -> Package_TO_SOT_SMD:SOT-23; symbol karta_stm-rescue:Q_NMOS_DGS-Device -> Device:Q_NMOS_GSD
- Q2: value Q_PMOS_DGS -> BSS84AKW.115; footprint Package_TO_SOT_SMD:SOT-23W_Handsoldering -> Package_TO_SOT_SMD:SOT-23; symbol karta_stm-rescue:Q_PMOS_DGS-Device -> Device:Q_NMOS_GSD
- R32, R33, R34, R35, R36, R37, R38, R39, R40, R41, R42, R43, R44, R45, R46, R47: footprint Resistor_SMD:R_1206_3216Metric_Pad1.42x1.75mm_HandSolder -> Resistor_SMD:R_0805_2012Metric
Connections:
- net GND: now also Q12.2 (S), Q15.2 (S), Q3.2 (S), Q6.2 (S), Q9.2 (S); no longer Q12.3 (S), Q15.3 (S), Q3.3 (S), Q6.3 (S), Q9.3 (S)
- net OUT_0: now also Q2.3 (D), Q3.3 (D); no longer Q2.1 (D), Q3.1 (D)
- net OUT_1: now also Q8.3 (D), Q9.3 (D); no longer Q8.1 (D), Q9.1 (D)
- net OUT_2: now also Q11.3 (D), Q12.3 (D); no longer Q11.1 (D), Q12.1 (D)
- net OUT_3: now also Q14.3 (D), Q15.3 (D); no longer Q14.1 (D), Q15.1 (D)
- net OUT_4: now also Q5.3 (D), Q6.3 (D); no longer Q5.1 (D), Q6.1 (D)
- net at R36.2: now also Q2.2 (S); no longer Q2.3 (S)
- net at Q1.3 (C), R33.2: now also Q2.1 (G), Q3.1 (G); no longer Q2.2 (G), Q3.2 (G)
- net at R41.2: now also Q8.2 (S); no longer Q8.3 (S)
- net at Q7.3 (C), R40.2: now also Q8.1 (G), Q9.1 (G); no longer Q8.2 (G), Q9.2 (G)
- net at R44.2: now also Q11.2 (S); no longer Q11.3 (S)
- net at Q10.3 (C), R43.2: now also Q11.1 (G), Q12.1 (G); no longer Q11.2 (G), Q12.2 (G)
- net at R47.2: now also Q14.2 (S); no longer Q14.3 (S)
- net at Q13.3 (C), R46.2: now also Q14.1 (G), Q15.1 (G); no longer Q14.2 (G), Q15.2 (G)
- net at R38.2: now also Q5.2 (S); no longer Q5.3 (S)
- net at Q4.3 (C), R37.2: now also Q5.1 (G), Q6.1 (G); no longer Q5.2 (G), Q6.2 (G)
Changed lines of the file:
@@
 F 0 "R32" V 493 1550 50  0000 C CNN
 F 1 "100R" V 584 1550 50  0000 C CNN
-F 2 "Resistor_SMD:R_1206_3216Metric_Pad1.42x1.75mm_HandSolder" V 630 1550 50  0001 C CNN
+F 2 "Resistor_SMD:R_0805_2012Metric" V 630 1550 50  0001 C CNN
 F 3 "~" H 700 1550 50  0001 C CNN
 	1    700  1550
@@
 F 0 "R36" H 1770 896 50  0000 L CNN
 F 1 "10k" H 1770 805 50  0000 L CNN
-F 2 "Resistor_SMD:R_1206_3216Metric_Pad1.42x1.75mm_HandSolder" V 1630 850 50  0001 C CNN
+F 2 "Resistor_SMD:R_0805_2012Metric" V 1630 850 50  0001 C CNN
 F 3 "~" H 1700 850 50  0001 C CNN
 	1    1700 850
@@
 	1700 1800 1700 1950
 $Comp
-L karta_stm-rescue:Q_PMOS_DGS-Device Q2
+L Device:Q_NMOS_GSD Q2
 U 1 1 5FA2941B
 P 1600 1200
 F 0 "Q2" H 1805 1246 50  0000 L CNN
-F 1 "Q_PMOS_DGS" H 1805 1155 50  0000 L CNN
-F 2 "Package_TO_SOT_SMD:SOT-23W_Handsoldering" H 1800 1300 50  0001 C CNN
+F 1 "BSS84AKW.115" H 1805 1155 50  0000 L CNN
+F 2 "Package_TO_SOT_SMD:SOT-23" H 1800 1300 50  0001 C CNN
 F 3 "~" H 1600 1200 50  0001 C CNN
 	1    1600 1200
@@
 $EndComp
 $Comp
-L karta_stm-rescue:Q_NMOS_DGS-Device Q3
+L Device:Q_NMOS_GSD Q3
 U 1 1 5FA2A75C
 P 1600 1600
 F 0 "Q3" H 1804 1646 50  0000 L CNN
-F 1 "Q_NMOS_DGS" H 1804 1555 50  0000 L CNN
-F 2 "Package_TO_SOT_SMD:SOT-23W_Handsoldering" H 1800 1700 50  0001 C CNN
+F 1 "BSS138W" H 1804 1555 50  0000 L CNN
+F 2 "Package_TO_SOT_SMD:SOT-23" H 1800 1700 50  0001 C CNN
 F 3 "~" H 1600 1600 50  0001 C CNN
 	1    1600 1600
@@
 F 0 "R41" H 4470 946 50  0000 L CNN
 F 1 "10k" H 4470 855 50  0000 L CNN
-F 2 "Resistor_SMD:R_1206_3216Metric_Pad1.42x1.75mm_HandSolder" V 4330 900 50  0001 C CNN
+F 2 "Resistor_SMD:R_0805_2012Metric" V 4330 900 50  0001 C CNN
 F 3 "~" H 4400 900 50  0001 C CNN
 	1    4400 900
@@
 	4100 1450 4100 1250
 $Comp
-L karta_stm-rescue:Q_PMOS_DGS-Device Q8
+L Device:Q_PMOS_GSD Q8
 U 1 1 5FA2E69C
 P 4300 1250
 F 0 "Q8" H 4505 1296 50  0000 L CNN
-F 1 "Q_PMOS_DGS" H 4505 1205 50  0000 L CNN
-F 2 "Package_TO_SOT_SMD:SOT-23W_Handsoldering" H 4500 1350 50  0001 C CNN
+F 1 "BSS84AKW.115" H 4505 1205 50  0000 L CNN
+F 2 "Package_TO_SOT_SMD:SOT-23" H 4500 1350 50  0001 C CNN
 F 3 "~" H 4300 1250 50  0001 C CNN
 	1    4300 1250
@@
 $EndComp
 $Comp
-L karta_stm-rescue:Q_NMOS_DGS-Device Q9
+L Device:Q_NMOS_GSD Q9
 U 1 1 5FA2E6A2
 P 4300 1650
 F 0 "Q9" H 4504 1696 50  0000 L CNN
-F 1 "Q_NMOS_DGS" H 4504 1605 50  0000 L CNN
-F 2 "Package_TO_SOT_SMD:SOT-23W_Handsoldering" H 4500 1750 50  0001 C CNN
+F 1 "BSS138W" H 4504 1605 50  0000 L CNN
+F 2 "Package_TO_SOT_SMD:SOT-23" H 4500 1750 50  0001 C CNN
 F 3 "~" H 4300 1650 50  0001 C CNN
 	1    4300 1650
@@
 F 0 "R44" H 7420 896 50  0000 L CNN
 F 1 "10k" H 7420 805 50  0000 L CNN
-F 2 "Resistor_SMD:R_1206_3216Metric_Pad1.42x1.75mm_HandSolder" V 7280 850 50  0001 C CNN
+F 2 "Resistor_SMD:R_0805_2012Metric" V 7280 850 50  0001 C CNN
 F 3 "~" H 7350 850 50  0001 C CNN
 	1    7350 850
@@
 	7350 1800 7350 1950
 $Comp
-L karta_stm-rescue:Q_PMOS_DGS-Device Q11
+L Device:Q_PMOS_GSD Q11
 U 1 1 5FA2EC34
 P 7250 1200
 F 0 "Q11" H 7455 1246 50  0000 L CNN
-F 1 "Q_PMOS_DGS" H 7455 1155 50  0000 L CNN
-F 2 "Package_TO_SOT_SMD:SOT-23W_Handsoldering" H 7450 1300 50  0001 C CNN
+F 1 "BSS84AKW.115" H 7455 1155 50  0000 L CNN
+F 2 "Package_TO_SOT_SMD:SOT-23" H 7450 1300 50  0001 C CNN
 F 3 "~" H 7250 1200 50  0001 C CNN
 	1    7250 1200
@@
 $EndComp
 $Comp
-L karta_stm-rescue:Q_NMOS_DGS-Device Q12
+L Device:Q_NMOS_GSD Q12
 U 1 1 5FA2EC3A
 P 7250 1600
 F 0 "Q12" H 7454 1646 50  0000 L CNN
-F 1 "Q_NMOS_DGS" H 7454 1555 50  0000 L CNN
-F 2 "Package_TO_SOT_SMD:SOT-23W_Handsoldering" H 7450 1700 50  0001 C CNN
+F 1 "BSS138W" H 7454 1555 50  0000 L CNN
+F 2 "Package_TO_SOT_SMD:SOT-23" H 7450 1700 50  0001 C CNN
 F 3 "~" H 7250 1600 50  0001 C CNN
 	1    7250 1600
@@
 F 0 "R38" H 2420 2696 50  0000 L CNN
 F 1 "10k" H 2420 2605 50  0000 L CNN
-F 2 "Resistor_SMD:R_1206_3216Metric_Pad1.42x1.75mm_HandSolder" V 2280 2650 50  0001 C CNN
+F 2 "Resistor_SMD:R_0805_2012Metric" V 2280 2650 50  0001 C CNN
 F 3 "~" H 2350 2650 50  0001 C CNN
 	1    2350 2650
@@
 	2350 3600 2350 3750
 $Comp
-L karta_stm-rescue:Q_PMOS_DGS-Device Q5
+L Device:Q_PMOS_GSD Q5
 U 1 1 5FA36A4F
 P 2250 3000
 F 0 "Q5" H 2455 3046 50  0000 L CNN
-F 1 "Q_PMOS_DGS" H 2455 2955 50  0000 L CNN
-F 2 "Package_TO_SOT_SMD:SOT-23W_Handsoldering" H 2450 3100 50  0001 C CNN
+F 1 "BSS84AKW.115" H 2455 2955 50  0000 L CNN
+F 2 "Package_TO_SOT_SMD:SOT-23" H 2450 3100 50  0001 C CNN
 F 3 "~" H 2250 3000 50  0001 C CNN
 	1    2250 3000
@@
 $EndComp
 $Comp
-L karta_stm-rescue:Q_NMOS_DGS-Device Q6
+L Device:Q_NMOS_GSD Q6
 U 1 1 5FA36A55
 P 2250 3400
 F 0 "Q6" H 2454 3446 50  0000 L CNN
-F 1 "Q_NMOS_DGS" H 2454 3355 50  0000 L CNN
-F 2 "Package_TO_SOT_SMD:SOT-23W_Handsoldering" H 2450 3500 50  0001 C CNN
+F 1 "BSS138W" H 2454 3355 50  0000 L CNN
+F 2 "Package_TO_SOT_SMD:SOT-23" H 2450 3500 50  0001 C CNN
 F 3 "~" H 2250 3400 50  0001 C CNN
 	1    2250 3400
@@
 Connection ~ 9950 1500
 $Comp
-L karta_stm-rescue:Q_NMOS_DGS-Device Q15
+L Device:Q_NMOS_GSD Q15
 U 1 1 5FA318F3
 P 9850 1700
 F 0 "Q15" H 10054 1746 50  0000 L CNN
-F 1 "Q_NMOS_DGS" H 10054 1655 50  0000 L CNN
-F 2 "Package_TO_SOT_SMD:SOT-23W_Handsoldering" H 10050 1800 50  0001 C CNN
+F 1 "BSS138W" H 10054 1655 50  0000 L CNN
+F 2 "Package_TO_SOT_SMD:SOT-23" H 10050 1800 50  0001 C CNN
 F 3 "~" H 9850 1700 50  0001 C CNN
 	1    9850 1700
@@
 $EndComp
 $Comp
-L karta_stm-rescue:Q_PMOS_DGS-Device Q14
+L Device:Q_PMOS_GSD Q14
 U 1 1 5FA318ED
 P 9850 1300
 F 0 "Q14" H 10055 1346 50  0000 L CNN
-F 1 "Q_PMOS_DGS" H 10055 1255 50  0000 L CNN
-F 2 "Package_TO_SOT_SMD:SOT-23W_Handsoldering" H 10050 1400 50  0001 C CNN
+F 1 "BSS84AKW.115" H 10055 1255 50  0000 L CNN
+F 2 "Package_TO_SOT_SMD:SOT-23" H 10050 1400 50  0001 C CNN
 F 3 "~" H 9850 1300 50  0001 C CNN
 	1    9850 1300
@@
 F 0 "R47" H 10020 996 50  0000 L CNN
 F 1 "10k" H 10020 905 50  0000 L CNN
-F 2 "Resistor_SMD:R_1206_3216Metric_Pad1.42x1.75mm_HandSolder" V 9880 950 50  0001 C CNN
+F 2 "Resistor_SMD:R_0805_2012Metric" V 9880 950 50  0001 C CNN
 F 3 "~" H 9950 950 50  0001 C CNN
 	1    9950 950
@@
 F 0 "R35" V 1243 4400 50  0000 C CNN
 F 1 "10k" V 1334 4400 50  0000 C CNN
-F 2 "Resistor_SMD:R_1206_3216Metric_Pad1.42x1.75mm_HandSolder" V 1380 4400 50  0001 C CNN
+F 2 "Resistor_SMD:R_0805_2012Metric" V 1380 4400 50  0001 C CNN
 F 3 "~" H 1450 4400 50  0001 C CNN
 	1    1450 4400
@@
 F 0 "F2" V 953 4400 50  0000 C CNN
 F 1 "100mA" V 1044 4400 50  0000 C CNN
-F 2 "Fuse:Fuse_2920_7451Metric_Pad2.10x5.45mm_HandSolder" V 1080 4400 50  0001 C CNN
+F 2 "Fuse:Fuse_1206_3216Metric_Pad1.42x1.75mm_HandSolder" V 1080 4400 50  0001 C CNN
 F 3 "~" H 1150 4400 50  0001 C CNN
 	1    1150 4400
@@
 F 0 "R40" H 3920 1346 50  0000 L CNN
 F 1 "10k" H 3920 1255 50  0000 L CNN
-F 2 "Resistor_SMD:R_1206_3216Metric_Pad1.42x1.75mm_HandSolder" V 3780 1300 50  0001 C CNN
+F 2 "Resistor_SMD:R_0805_2012Metric" V 3780 1300 50  0001 C CNN
 F 3 "~" H 3850 1300 50  0001 C CNN
 	1    3850 1300
@@
 F 0 "R43" H 6870 1296 50  0000 L CNN
 F 1 "10k" H 6870 1205 50  0000 L CNN
-F 2 "Resistor_SMD:R_1206_3216Metric_Pad1.42x1.75mm_HandSolder" V 6730 1250 50  0001 C CNN
+F 2 "Resistor_SMD:R_0805_2012Metric" V 6730 1250 50  0001 C CNN
 F 3 "~" H 6800 1250 50  0001 C CNN
 	1    6800 1250
@@
 F 0 "R46" H 9470 1346 50  0000 L CNN
 F 1 "10k" H 9470 1255 50  0000 L CNN
-F 2 "Resistor_SMD:R_1206_3216Metric_Pad1.42x1.75mm_HandSolder" V 9330 1300 50  0001 C CNN
+F 2 "Resistor_SMD:R_0805_2012Metric" V 9330 1300 50  0001 C CNN
 F 3 "~" H 9400 1300 50  0001 C CNN
 	1    9400 1300
@@
 F 0 "R39" V 3607 1650 50  0000 C CNN
 F 1 "100R" V 3516 1650 50  0000 C CNN
-F 2 "Resistor_SMD:R_1206_3216Metric_Pad1.42x1.75mm_HandSolder" V 3330 1650 50  0001 C CNN
+F 2 "Resistor_SMD:R_0805_2012Metric" V 3330 1650 50  0001 C CNN
 F 3 "~" H 3400 1650 50  0001 C CNN
 	1    3400 1650
@@
 F 0 "R42" V 6143 1600 50  0000 C CNN
 F 1 "100R" V 6234 1600 50  0000 C CNN
-F 2 "Resistor_SMD:R_1206_3216Metric_Pad1.42x1.75mm_HandSolder" V 6280 1600 50  0001 C CNN
+F 2 "Resistor_SMD:R_0805_2012Metric" V 6280 1600 50  0001 C CNN
 F 3 "~" H 6350 1600 50  0001 C CNN
 	1    6350 1600
@@
 F 0 "R45" V 8743 1650 50  0000 C CNN
 F 1 "100R" V 8834 1650 50  0000 C CNN
-F 2 "Resistor_SMD:R_1206_3216Metric_Pad1.42x1.75mm_HandSolder" V 8880 1650 50  0001 C CNN
+F 2 "Resistor_SMD:R_0805_2012Metric" V 8880 1650 50  0001 C CNN
 F 3 "~" H 8950 1650 50  0001 C CNN
 	1    8950 1650
@@
 F 0 "R37" H 1870 3096 50  0000 L CNN
 F 1 "10k" H 1870 3005 50  0000 L CNN
-F 2 "Resistor_SMD:R_1206_3216Metric_Pad1.42x1.75mm_HandSolder" V 1730 3050 50  0001 C CNN
+F 2 "Resistor_SMD:R_0805_2012Metric" V 1730 3050 50  0001 C CNN
 F 3 "~" H 1800 3050 50  0001 C CNN
 	1    1800 3050
@@
 F 0 "R34" V 1143 3400 50  0000 C CNN
 F 1 "100R" V 1234 3400 50  0000 C CNN
-F 2 "Resistor_SMD:R_1206_3216Metric_Pad1.42x1.75mm_HandSolder" V 1280 3400 50  0001 C CNN
+F 2 "Resistor_SMD:R_0805_2012Metric" V 1280 3400 50  0001 C CNN
 F 3 "~" H 1350 3400 50  0001 C CNN
 	1    1350 3400
@@
 F 0 "R33" H 1220 1246 50  0000 L CNN
 F 1 "10k" H 1220 1155 50  0000 L CNN
-F 2 "Resistor_SMD:R_1206_3216Metric_Pad1.42x1.75mm_HandSolder" V 1080 1200 50  0001 C CNN
+F 2 "Resistor_SMD:R_0805_2012Metric" V 1080 1200 50  0001 C CNN
 F 3 "~" H 1150 1200 50  0001 C CNN
 	1    1150 1200
