File: karta_stm/karta_stm.kicad_pcb (KiCad board)
At the start: 2 copper layers, 100.5 x 62.9 mm, 137 parts, among them J1 Conn_01x02_Female, J2 Conn_01x06_Male, J3 Conn_01x05_Female, J4 Conn_01x02_Female, J5 Conn_01x05_Female, J6 Conn_01x04_Female, J7 Conn_01x03_Male, Q1 BC817, Q10 BC817, Q11 Q_PMOS_DGS, Q12 Q_NMOS_DGS, Q13 BC817, Q14 Q_PMOS_DGS, Q15 Q_NMOS_DGS, Q2 Q_PMOS_DGS, Q3 Q_NMOS_DGS, Q4 BC817, Q5 Q_PMOS_DGS, Q6 Q_NMOS_DGS, Q7 BC817, Q8 Q_PMOS_DGS, Q9 Q_NMOS_DGS, SW1 SW_Push, U1 STM32L4P5RET6, U10 EL817, U11 EL817, U12 EL817, U13 EL817, U2 MCP2562-H-SN, U3 LM2596S-5, U4 LD1117S33TR_SOT223, U5 MCP6001x-LT, U6 MCP6001x-LT, U7 MCP6001x-LT, U8 MCP6001x-LT, U9 MCP6001x-LT, Y1 16MHz

Commit message: Update pcb
Parts:
- removed G***: LOGO, Logos:PUTM_LOGO_26mm
- removed G***: LOGO, Logos:SignatureBox25mm
- C1, C2: footprint Capacitor_SMD:C_0805_2012Metric_Pad1.15x1.40mm_HandSolder -> Capacitor_SMD:C_0805_2012Metric
- C10, C12, C18, C19, C20, C21, C22, C3: footprint Capacitor_SMD:C_1206_3216Metric_Pad1.42x1.75mm_HandSolder -> Capacitor_SMD:C_1206_3216Metric
- C11: footprint Capacitor_SMD:C_1206_3216Metric_Pad1.42x1.75mm_HandSolder -> Capacitor_SMD:CP_Elec_4x5.7
- C9: footprint Capacitor_Tantalum_SMD:CP_EIA-6032-15_Kemet-U_Pad2.25x2.35mm_HandSolder -> Capacitor_Tantalum_SMD:CP_EIA-6032-15_Kemet-U
- D11, D12: footprint Diode_SMD:D_1210_3225Metric_Pad1.42x2.65mm_HandSolder -> Diode_SMD:D_1210_3225Metric
- D3: value D_Schottky -> SS24T3G
- F1, F2: footprint Fuse:Fuse_2920_7451Metric_Pad2.10x5.45mm_HandSolder -> Fuse:Fuse_1206_3216Metric_Pad1.42x1.75mm_HandSolder
- Q11, Q14, Q2, Q5, Q8: value Q_PMOS_DGS -> BSS84AKW.115; footprint Package_TO_SOT_SMD:SOT-23W_Handsoldering -> Package_TO_SOT_SMD:SOT-23
- Q12, Q15, Q3, Q6, Q9: value Q_NMOS_DGS -> BSS138W; footprint Package_TO_SOT_SMD:SOT-23W_Handsoldering -> Package_TO_SOT_SMD:SOT-23
- R1: footprint Resistor_SMD:R_1206_3216Metric_Pad1.42x1.75mm_HandSolder -> Resistor_SMD:R_1206_3216Metric
- R10, R11, R12, R13, R14, R15, R16, R17, R18, R19, R2, R20, R21, R22, R23, R24, R25, R26, R27, R28, R29, R3, R30, R31, R32, R33, R34, R35, R36, R37, R38, R39, R4, R40, R42, R43, R44, R45, R46, R47, R48, R5, R6, R7, R8, R9: footprint Resistor_SMD:R_1206_3216Metric_Pad1.42x1.75mm_HandSolder -> Resistor_SMD:R_0805_2012Metric
- R41: value 100k -> 10k; footprint Resistor_SMD:R_1206_3216Metric_Pad1.42x1.75mm_HandSolder -> Resistor_SMD:R_0805_2012Metric
- R49: value 1kOhm -> 5kOhm; footprint Resistor_SMD:R_1206_3216Metric_Pad1.42x1.75mm_HandSolder -> Resistor_SMD:R_0805_2012Metric
- SW1: footprint Button_Switch_SMD:SW_Push_1P1T_NO_6x6mm_H9.5mm -> Resistor_SMD:R_0805_2012Metric
- U4: value LD1117S33TR_SOT223 -> LM1117-3.3
- moved Q14 1.07 mm to (107.2, 76.3)
- moved Q5 1.07 mm to (107.3, 69.7), turned to 180 degrees
- moved Q15 1.02 mm to (103.1, 75.1), turned to 270 degrees
- moved Q8 0.97 mm to (108.3, 90.4)
- moved Q9 0.90 mm to (102.5, 89.4), turned to 270 degrees
- moved Q12 0.85 mm to (101.2, 82.3), turned to 270 degrees
- moved R31 0.85 mm to (158.6, 64.1)
- moved Q2 0.76 mm to (107.7, 98.2)
- moved U13 0.51 mm to (154.7, 58.1)
- moved Q3 0.42 mm to (101.9, 97.2), turned to 270 degrees
- moved R49 0.19 mm to (149.8, 106.3)
- moved Q6 0.13 mm to (101.1, 67.9), turned to 0 degrees
Connections:
- C15 pad 2: Net-(C15-Pad2) -> GND
- C16 pad 2: Net-(C15-Pad2) -> GND
- Q11 pad 1: OUT_2 -> Net-(Q10-Pad3)
- Q11 pad 2: Net-(Q10-Pad3) -> Net-(Q11-Pad2)
- Q11 pad 3: Net-(Q11-Pad3) -> OUT_2
- Q12 pad 1: OUT_2 -> Net-(Q10-Pad3)
- Q12 pad 2: Net-(Q10-Pad3) -> GND
- Q12 pad 3: GND -> OUT_2
- Q14 pad 1: OUT_3 -> Net-(Q13-Pad3)
- Q14 pad 2: Net-(Q13-Pad3) -> Net-(Q14-Pad2)
- Q14 pad 3: Net-(Q14-Pad3) -> OUT_3
- Q15 pad 1: OUT_3 -> Net-(Q13-Pad3)
- Q15 pad 2: Net-(Q13-Pad3) -> GND
- Q15 pad 3: GND -> OUT_3
- Q2 pad 1: OUT_0 -> Net-(Q1-Pad3)
- Q2 pad 2: Net-(Q1-Pad3) -> Net-(Q2-Pad2)
- Q2 pad 3: Net-(Q2-Pad3) -> OUT_0
- Q3 pad 1: OUT_0 -> Net-(Q1-Pad3)
- Q3 pad 2: Net-(Q1-Pad3) -> GND
- Q3 pad 3: GND -> OUT_0
- Q5 pad 1: OUT_4 -> Net-(Q4-Pad3)
- Q5 pad 2: Net-(Q4-Pad3) -> Net-(Q5-Pad2)
- Q5 pad 3: Net-(Q5-Pad3) -> OUT_4
- Q6 pad 1: OUT_4 -> Net-(Q4-Pad3)
- Q6 pad 2: Net-(Q4-Pad3) -> GND
- Q6 pad 3: GND -> OUT_4
- Q8 pad 1: OUT_1 -> Net-(Q7-Pad3)
- Q8 pad 2: Net-(Q7-Pad3) -> Net-(Q8-Pad2)
- Q8 pad 3: Net-(Q8-Pad3) -> OUT_1
- Q9 pad 1: OUT_1 -> Net-(Q7-Pad3)
- Q9 pad 2: Net-(Q7-Pad3) -> GND
- Q9 pad 3: GND -> OUT_1
- R36 pad 2: Net-(Q2-Pad3) -> Net-(Q2-Pad2)
- R38 pad 2: Net-(Q5-Pad3) -> Net-(Q5-Pad2)
- R41 pad 2: Net-(Q8-Pad3) -> Net-(Q8-Pad2)
- R44 pad 2: Net-(Q11-Pad3) -> Net-(Q11-Pad2)
- R47 pad 2: Net-(Q14-Pad3) -> Net-(Q14-Pad2)
- U1 pad 15: Net-(U1-Pad15) -> (no net)
- U1 pad 16: Net-(U1-Pad16) -> (no net)
- U1 pad 17: Net-(U1-Pad17) -> (no net)
- U1 pad 20: Net-(U1-Pad20) -> (no net)
- U1 pad 21: Net-(U1-Pad21) -> (no net)
- U1 pad 22: Net-(U1-Pad22) -> (no net)
- U1 pad 23: Net-(U1-Pad23) -> (no net)
- U1 pad 26: Net-(U1-Pad26) -> (no net)
- U1 pad 29: Net-(U1-Pad29) -> (no net)
- U1 pad 3: Net-(U1-Pad3) -> (no net)
- U1 pad 30: Net-(U1-Pad30) -> (no net)
- U1 pad 33: Net-(U1-Pad33) -> (no net)
- U1 pad 34: Net-(U1-Pad34) -> (no net)
- U1 pad 35: Net-(U1-Pad35) -> (no net)
- U1 pad 36: Net-(U1-Pad36) -> (no net)
- U1 pad 37: Net-(U1-Pad37) -> (no net)
- U1 pad 38: Net-(U1-Pad38) -> (no net)
- U1 pad 39: Net-(U1-Pad39) -> (no net)
- U1 pad 4: Net-(U1-Pad4) -> (no net)
- U1 pad 40: Net-(U1-Pad40) -> (no net)
- U1 pad 50: Net-(U1-Pad50) -> (no net)
- U1 pad 53: Net-(U1-Pad53) -> (no net)
- U1 pad 54: Net-(U1-Pad54) -> (no net)
- U1 pad 56: Net-(U1-Pad56) -> (no net)
- U1 pad 57: Net-(U1-Pad57) -> (no net)
- U1 pad 59: Net-(U1-Pad59) -> (no net)
- U4 pad 1: Net-(C15-Pad2) -> GND
Routing:
- net GND: track 700.3 -> 749.8 mm, vias 65 -> 64
- net Net-(C15-Pad2): track 33.1 -> 0.00 mm
- net Net-(Q11-Pad3): track 7.81 -> 0.00 mm
- net Net-(Q8-Pad3): track 6.90 -> 0.00 mm
- net Net-(Q2-Pad3): track 6.81 -> 0.00 mm
- net Net-(Q14-Pad3): track 6.68 -> 0.00 mm
- net OUT_3: track 18.1 -> 12.0 mm
- net NRST: track 60.4 -> 54.2 mm
- net Net-(Q4-Pad3): track 22.5 -> 16.8 mm
- net Net-(Q10-Pad3): track 12.3 -> 17.8 mm
- net Net-(Q5-Pad2): track 0.00 -> 5.42 mm
- net Net-(Q14-Pad2): track 0.00 -> 5.14 mm
- net Net-(Q5-Pad3): track 5.12 -> 0.00 mm
- net OUT_0: track 26.9 -> 22.0 mm
- net Net-(Q11-Pad2): track 0.00 -> 4.75 mm
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